Commit message: Fix error 'Could not load resource ...hokuyo.dae' closes #1

File: urdf/dumpster.xacro (robot description, xacro)
@@ -250,5 +250,5 @@
       <origin xyz="0.0 0 0" rpy="0 0 0"/>
       <geometry>
-         <mesh filename="package://udacity_bot/meshes/hokuyo.dae"/>
+         <mesh filename="package://dumpster/meshes/hokuyo.dae"/>
       </geometry>
     </visual>
